Commit message: update piper_description folder from agilexrobotics/piper_ros

File: arm/piper_description/urdf/piper_description.urdf (robot description, URDF)
Before this commit: robot piper, 11 links, 10 joints
Joints:
- joint joint1: limit lower=-2.618 upper=2.168 effort=100 velocity=5 -> lower=-2.618 upper=2.618 effort=100 velocity=5

File: arm/piper_description/urdf/piper_description.xacro (robot description, xacro)
@@ -4,12 +4,12 @@
   xmlns:xacro="http://ros.org/wiki/xacro">
 <!-- world -->
-  <link name="world"/>
+  <!-- <link name="world"/>
   <joint name="fixed_base_joint" type="fixed">
       <parent link="world"/>
       <child link="base_link"/>
-  </joint>
+  </joint> -->
 <!-- piper -->
 <link
-    name="base_link">
+    name="arm_base">
     <inertial>
       <origin
@@ -97,5 +97,5 @@
       rpy="0 0 0" />
     <parent
-      link="base_link" />
+      link="arm_base" />
     <child
       link="link1" />
